File: Sensors.kicad_pcb (KiCad board)
At the start: 4 copper layers, 8 parts, among them U01 BMI270, U02 BMM150

Commit message: with layout, ready for review
Parts:
- added G***: LOGO, LOGO, F.Cu at (105.8, 48.0)
- added J1: Conn_01x06_Male, Connector_PinSocket_2.54mm:PinSocket_1x06_P2.54mm_Vertical, F.Cu at (101.8, 48.9)
- moved C2 15.4 mm to (90.3, 56.0), turned to 180 degrees
- moved C1 15.4 mm to (90.3, 52.5), turned to 180 degrees
- moved R1 15.3 mm to (100.1, 52.5)
- moved C4 14.6 mm to (104.6, 55.9)
- moved U01 14.6 mm to (100.1, 56.3)
- moved C3 14.4 mm to (104.6, 52.5)
- moved U02 13.6 mm to (94.5, 56.9)
- moved R2 13.4 mm to (94.8, 52.5)
Connections:
- net SDA_IMU renamed 3.3V
Routing:
- net Net-(U01-Pad2): track 1.60 -> 12.9 mm
- net GND: track 19.2 -> 9.50 mm, vias 5 -> 4
- net 3.3V: track 38.1 -> 28.3 mm, vias 3 -> 5
- net Net-(U01-Pad3): track 3.03 -> 12.1 mm, vias 0 -> 1
- net Net-(U01-Pad14): track 4.33 -> 10.2 mm
- net Net-(U01-Pad13): track 3.39 -> 8.02 mm
- added copper zone on In2.Cu, net 3.3V
- added copper zone on F.Cu, net GND
- added copper zone on In1.Cu, net GND
Other:
- board outline added: 20.8 x 14.3 mm
- board text added: "3.3V"
- board text added: "BB8"
- board text added: "E.Nutt"
- board text added: "GND"
- board text added: "SCK"
- board text added: "SCL"
- board text added: "SDA"
- board text added: "SDI"
