File: Sensors.kicad_sch (KiCad schematic)
At the start: 7 parts

Commit message: 01_14 edits
Parts:
- removed R?: 10k, Resistor_SMD:R_0603_1608Metric, symbol mainboard:R-US_R0603
- added R1, R2: 10k, Resistor_SMD:R_0603_1608Metric, symbol mainboard:R-US_R0603
- U01: renamed from U?; footprint mainboard:BMI270 -> Sensor_Motion:XDCR_BMI270
- U02: renamed from U?; footprint mainboard:BMM150 -> Sensor_Motion:XDCR_BMM150
- gave numbers to parts that had none: 4
Connections:
- net 3.3V: now also R1.1, R2.1
- net GND: now also U01.1 (SDO)
- net SCL_IMU: no longer names the net of U01.13 (SCX)
- net SCL_IMU: now also R1.2
- net SDA_IMU: no longer names the net of U01.14 (SDX)
- net SDA_IMU: now also R2.2

Commit message: with layout, ready for review
Parts:
- added J1: Conn_01x06_Male, symbol Connector:Conn_01x06_Male
Connections:
- net 3.3V: now also J1.6 (Pin_6)
- net GND: now also J1.5 (Pin_5)
- net at U01.3 (ASCX), U02.A3 (SCK): now also J1.3 (Pin_3)
- net at U01.2 (ASDX), U02.B4 (SDI): now also J1.4 (Pin_4)
- net at R1.2, U01.13 (SCX): now also J1.1 (Pin_1)
- net at R2.2, U01.14 (SDX): now also J1.2 (Pin_2)
Other:
- moved on the sheet: R1, R2
